File: W25Q-BRD.kicad_pcb (KiCad board)
At the start: 2 copper layers, 16 x 23 mm, 9 parts, among them J1 QSPI, U1 W25Q128JVSIQ

Commit message: Added alternative footprint for WSOT-8 version of the chip.
Parts:
- added U2: W25Q128JVPIQ, Package_SON:WSON-8-1EP_6x5mm_P1.27mm_EP3.4x4.3mm, F.Cu at (141.0, 101.0)
Routing:
- net +3.3V: track 26.4 -> 27.5 mm
- net /IO0: track 15.2 -> 16.2 mm
- net /CLK: track 16.3 -> 17.2 mm
- net /IO3: track 15.3 -> 16.2 mm
- net GND: track 0.00 -> 0.90 mm
- net /IO1: track 6.06 -> 6.96 mm
- net /NCS: track 7.67 -> 8.57 mm
- net /IO2: track 7.25 -> 8.15 mm
